File: step_down.sch (KiCad schematic (older format))
At the start: 12 parts, among them U3 MC34063AD

Commit message: update
Parts:
- removed R11, R12, R13: 3R3, Resistor_SMD:R_0603_1608Metric_Pad1.05x0.95mm_HandSolder, symbol Device:R
- added C10: 100u, symbol Device:CP
- added C11: 22u, symbol Device:CP
- added L2: 1u, symbol Device:L
- added U4: AMS1117-3.3, Package_TO_SOT_SMD:SOT-223-3_TabPin2, symbol Regulator_Linear:AMS1117-3.3
- C5: value 220u -> 100u
- C6: value 100u -> 47u
- D1: value SS34 -> SS24
- L1: value 220u -> 1m
- R14: value 3R3 -> 2R7
- R15: value 6.8k -> 12k
- R16: value 11k -> 36k
Connections:
- net GND: now also C10.2, C11.2, U4.1 (GND)
- net VCC: now also C11.1, U4.2 (VO); no longer C5.1, L1.2, R16.1
- new net: C5.1, L1.2, L2.1, R16.1
- new net: C10.1, L2.2, U4.3 (VI)
Other:
- note added: "150mA"
- note added: "Tantium"
- note removed: "360mA"
Changed lines of the file:
@@
 P 3550 1850
 F 0 "R14" V 3600 2000 50  0000 C CNN
-F 1 "3R3" V 3550 1850 50  0000 C CNN
+F 1 "2R7" V 3550 1850 50  0000 C CNN
 F 2 "Resistor_SMD:R_0603_1608Metric_Pad1.05x0.95mm_HandSolder" V 3480 1850 50  0001 C CNN
 F 3 "~" H 3550 1850 50  0001 C CNN
@@
 P 4400 2650
 F 0 "L1" V 4590 2650 50  0000 C CNN
-F 1 "220u" V 4499 2650 50  0000 C CNN
+F 1 "1m" V 4499 2650 50  0000 C CNN
 F 2 "EFan:SMD,4.5x4x3.2mm Inductor" H 4400 2650 50  0001 C CNN
 F 3 "~" H 4400 2650 50  0001 C CNN
@@
 P 4600 2850
 F 0 "C5" H 4718 2896 50  0000 L CNN
-F 1 "220u" H 4718 2805 50  0000 L CNN
+F 1 "100u" H 4718 2805 50  0000 L CNN
 F 2 "Capacitor_SMD:CP_Elec_8x10" H 4638 2700 50  0001 C CNN
 F 3 "~" H 4600 2850 50  0001 C CNN
@@
 P 4100 2850
 F 0 "D1" V 4054 2929 50  0000 L CNN
-F 1 "SS34" V 4145 2929 50  0000 L CNN
+F 1 "SS24" V 4145 2929 50  0000 L CNN
 F 2 "Diode_SMD:D_SMA_Handsoldering" H 4100 2850 50  0001 C CNN
 F 3 "~" H 4100 2850 50  0001 C CNN
@@
 	4600 2650 4750 2650
 Connection ~ 4600 2650
-Text HLabel 4900 2650 2    50   Output ~ 0
+Text HLabel 6600 2650 2    50   Output ~ 0
 VCC
-Text Notes 2150 3900 0    50   ~ 0
+Text Notes 1650 4250 0    50   ~ 0
 I(min) = 21.6\n27V -> 3.3V\n\nIo  = 150mA \nIpk = 2Io = 300mA\nTon = 3.8u\n\nLmin = (21.6-0.8-3.3 / Ipk )* Ton\n        = 220u\n\nI'pk = 395mA\nRsc = 0.33 / I'pk = 0.838 about 1ohm
-$Comp
-L Device:R R13
-U 1 1 5DBE442D
-P 3550 1700
-F 0 "R13" V 3600 1850 50  0000 C CNN
-F 1 "3R3" V 3550 1700 50  0000 C CNN
-F 2 "Resistor_SMD:R_0603_1608Metric_Pad1.05x0.95mm_HandSolder" V 3480 1700 50  0001 C CNN
-F 3 "~" H 3550 1700 50  0001 C CNN
-	1    3550 1700
-	0    -1   -1   0
-$EndComp
-$Comp
-L Device:R R12
-U 1 1 5DBE47E1
-P 3550 1550
-F 0 "R12" V 3600 1700 50  0000 C CNN
-F 1 "3R3" V 3550 1550 50  0000 C CNN
-F 2 "Resistor_SMD:R_0603_1608Metric_Pad1.05x0.95mm_HandSolder" V 3480 1550 50  0001 C CNN
-F 3 "~" H 3550 1550 50  0001 C CNN
-	1    3550 1550
-	0    -1   -1   0
-$EndComp
-$Comp
-L Device:R R11
-U 1 1 5DBE4AED
-P 3550 1400
-F 0 "R11" V 3600 1550 50  0000 C CNN
-F 1 "3R3" V 3550 1400 50  0000 C CNN
-F 2 "Resistor_SMD:R_0603_1608Metric_Pad1.05x0.95mm_HandSolder" V 3480 1400 50  0001 C CNN
-F 3 "~" H 3550 1400 50  0001 C CNN
-	1    3550 1400
-	0    -1   -1   0
-$EndComp
-Wire Wire Line
-	3400 1400 3100 1400
-Wire Wire Line
-	3100 1400 3100 1550
-Connection ~ 3100 1850
-Wire Wire Line
-	4000 1850 4000 1700
-Wire Wire Line
-	4000 1400 3700 1400
-Connection ~ 4000 1850
-Wire Wire Line
-	3700 1550 4000 1550
-Connection ~ 4000 1550
-Wire Wire Line
-	4000 1550 4000 1400
-Wire Wire Line
-	3400 1550 3100 1550
-Connection ~ 3100 1550
-Wire Wire Line
-	3100 1550 3100 1700
-Wire Wire Line
-	3400 1700 3100 1700
-Connection ~ 3100 1700
-Wire Wire Line
-	3100 1700 3100 1850
-Wire Wire Line
-	3700 1700 4000 1700
-Connection ~ 4000 1700
-Wire Wire Line
-	4000 1700 4000 1550
 Text Notes 4300 2400 0    50   ~ 0
-360mA
+150mA
 $Comp
 L Device:R R15
@@
 P 3750 3250
 F 0 "R15" V 3543 3250 50  0000 C CNN
-F 1 "6.8k" V 3634 3250 50  0000 C CNN
+F 1 "12k" V 3634 3250 50  0000 C CNN
 F 2 "Resistor_SMD:R_0603_1608Metric_Pad1.05x0.95mm_HandSolder" V 3680 3250 50  0001 C CNN
 F 3 "~" H 3750 3250 50  0001 C CNN
@@
 P 4200 3250
 F 0 "R16" V 3993 3250 50  0000 C CNN
-F 1 "11k" V 4084 3250 50  0000 C CNN
+F 1 "36k" V 4084 3250 50  0000 C CNN
 F 2 "Resistor_SMD:R_0603_1608Metric_Pad1.05x0.95mm_HandSolder" V 4130 3250 50  0001 C CNN
 F 3 "~" H 4200 3250 50  0001 C CNN
@@
 Connection ~ 4750 2650
 Wire Wire Line
-	4750 2650 4900 2650
-Wire Wire Line
 	4050 3250 4000 3250
 Wire Wire Line
@@
 P 2700 2600
 F 0 "C6" H 2818 2646 50  0000 L CNN
-F 1 "100u" H 2818 2555 50  0000 L CNN
+F 1 "47u" H 2818 2555 50  0000 L CNN
 F 2 "Capacitor_SMD:CP_Elec_8x10" H 2738 2450 50  0001 C CNN
 F 3 "~" H 2700 2600 50  0001 C CNN
@@
 Wire Wire Line
 	2700 2250 3100 2250
+$Comp
+L Device:L L2
+U 1 1 5DBDF5D2
+P 5100 2650
+F 0 "L2" V 5290 2650 50  0000 C CNN
+F 1 "1u" V 5199 2650 50  0000 C CNN
+F 2 "" H 5100 2650 50  0001 C CNN
+F 3 "~" H 5100 2650 50  0001 C CNN
+	1    5100 2650
+	0    -1   -1   0
+$EndComp
+$Comp
+L Device:CP C10
+U 1 1 5DBDFDFE
+P 5350 2850
+F 0 "C10" H 5468 2896 50  0000 L CNN
+F 1 "100u" H 5468 2805 50  0000 L CNN
+F 2 "" H 5388 2700 50  0001 C CNN
+F 3 "~" H 5350 2850 50  0001 C CNN
+	1    5350 2850
+	1    0    0    -1
+$EndComp
+Wire Wire Line
+	5250 2650 5350 2650
+Wire Wire Line
+	5350 2650 5350 2700
+Wire Wire Line
+	4750 2650 4950 2650
+Wire Wire Line
+	4600 3050 5350 3050
+Wire Wire Line
+	5350 3050 5350 3000
+Connection ~ 4600 3050
+$Comp
+L Regulator_Linear:AMS1117-3.3 U4
+U 1 1 5DBE2BB8
+P 6000 2650
+F 0 "U4" H 6000 2892 50  0000 C CNN
+F 1 "AMS1117-3.3" H 6000 2801 50  0000 C CNN
+F 2 "Package_TO_SOT_SMD:SOT-223-3_TabPin2" H 6000 2850 50  0001 C CNN
+F 3 "http://www.advanced-monolithic.com/pdf/ds1117.pdf" H 6100 2400 50  0001 C CNN
+	1    6000 2650
+	1    0    0    -1
+$EndComp
+Wire Wire Line
+	6000 2950 6000 3050
+Wire Wire Line
+	5350 3050 6000 3050
+Connection ~ 5350 3050
+Wire Wire Line
+	5350 2650 5700 2650
+Connection ~ 5350 2650
+$Comp
+L Device:CP C11
+U 1 1 5DBE5DDC
+P 6400 2850
+F 0 "C11" H 6518 2896 50  0000 L CNN
+F 1 "22u" H 6518 2805 50  0000 L CNN
+F 2 "" H 6438 2700 50  0001 C CNN
+F 3 "~" H 6400 2850 50  0001 C CNN
+	1    6400 2850
+	1    0    0    -1
+$EndComp
+Wire Wire Line
+	6400 3000 6400 3050
+Wire Wire Line
+	6400 3050 6000 3050
+Connection ~ 6000 3050
+Wire Wire Line
+	6400 2700 6400 2650
+Wire Wire Line
+	6400 2650 6300 2650
+Wire Wire Line
+	6400 2650 6600 2650
+Connection ~ 6400 2650
+Text Notes 6350 3200 0    50   ~ 0
+Tantium
 $EndSCHEMATC

Commit message: production 2
Parts:
- added TP10: 5V, TestPoint:TestPoint_Loop_D2.50mm_Drill1.0mm, symbol Connector:TestPoint
- added TP11: 3.3V, TestPoint:TestPoint_Loop_D2.50mm_Drill1.0mm, symbol Connector:TestPoint
- added TP7: 28V Loop, TestPoint:TestPoint_Loop_D2.50mm_Drill1.0mm, symbol Connector:TestPoint
- added TP8: GND Loop, TestPoint:TestPoint_Loop_D2.50mm_Drill1.0mm, symbol Connector:TestPoint
- added TP9: 5VRAW, TestPoint:TestPoint_Loop_D2.50mm_Drill1.0mm, symbol Connector:TestPoint
- C10: footprint (none) -> EFan:C_Radial_D5.0mm_H7.0mm_P2.00mm
- C11: footprint (none) -> EFan:CP_EIA-3216-18_Kemet-A_Pad1.58x1.35mm_HandSolder
- C5: footprint Capacitor_SMD:CP_Elec_8x10 -> EFan:C_Radial_D5.0mm_H7.0mm_P2.00mm
- C6: footprint Capacitor_SMD:CP_Elec_8x10 -> EFan:CP_Elec_6.3x5.4
- L1: footprint EFan:SMD,4.5x4x3.2mm Inductor -> EFan:L_Radial_D7.0mm_P3.00mm
- L2: footprint (none) -> Inductor_SMD:L_0805_2012Metric_Pad1.15x1.40mm_HandSolder
Connections:
- net +28V: now also TP7.1
- net GND: now also TP8.1
- net VCC: now also TP11.1
- net Sensed28: now reaches R14.2, U3.1 (SwC), U3.7 (Ipk), U3.8 (DC)
- net at C5.1, L1.2, L2.1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: now also TP9.1
- net at C10.1, L2.2, U4.3 (VI): now also TP10.1
Changed lines of the file:
@@
 F 0 "L1" V 4590 2650 50  0000 C CNN
 F 1 "1m" V 4499 2650 50  0000 C CNN
-F 2 "EFan:SMD,4.5x4x3.2mm Inductor" H 4400 2650 50  0001 C CNN
+F 2 "EFan:L_Radial_D7.0mm_P3.00mm" H 4400 2650 50  0001 C CNN
 F 3 "~" H 4400 2650 50  0001 C CNN
 	1    4400 2650
@@
 F 0 "C5" H 4718 2896 50  0000 L CNN
 F 1 "100u" H 4718 2805 50  0000 L CNN
-F 2 "Capacitor_SMD:CP_Elec_8x10" H 4638 2700 50  0001 C CNN
+F 2 "EFan:C_Radial_D5.0mm_H7.0mm_P2.00mm" H 4638 2700 50  0001 C CNN
 F 3 "~" H 4600 2850 50  0001 C CNN
 	1    4600 2850
@@
 F 0 "C6" H 2818 2646 50  0000 L CNN
 F 1 "47u" H 2818 2555 50  0000 L CNN
-F 2 "Capacitor_SMD:CP_Elec_8x10" H 2738 2450 50  0001 C CNN
+F 2 "EFan:CP_Elec_6.3x5.4" H 2738 2450 50  0001 C CNN
 F 3 "~" H 2700 2600 50  0001 C CNN
 	1    2700 2600
@@
 F 0 "L2" V 5290 2650 50  0000 C CNN
 F 1 "1u" V 5199 2650 50  0000 C CNN
-F 2 "" H 5100 2650 50  0001 C CNN
+F 2 "Inductor_SMD:L_0805_2012Metric_Pad1.15x1.40mm_HandSolder" H 5100 2650 50  0001 C CNN
 F 3 "~" H 5100 2650 50  0001 C CNN
 	1    5100 2650
@@
 F 0 "C10" H 5468 2896 50  0000 L CNN
 F 1 "100u" H 5468 2805 50  0000 L CNN
-F 2 "" H 5388 2700 50  0001 C CNN
+F 2 "EFan:C_Radial_D5.0mm_H7.0mm_P2.00mm" H 5388 2700 50  0001 C CNN
 F 3 "~" H 5350 2850 50  0001 C CNN
 	1    5350 2850
@@
 F 0 "C11" H 6518 2896 50  0000 L CNN
 F 1 "22u" H 6518 2805 50  0000 L CNN
-F 2 "" H 6438 2700 50  0001 C CNN
+F 2 "EFan:CP_EIA-3216-18_Kemet-A_Pad1.58x1.35mm_HandSolder" H 6438 2700 50  0001 C CNN
 F 3 "~" H 6400 2850 50  0001 C CNN
 	1    6400 2850
@@
 Text Notes 6350 3200 0    50   ~ 0
 Tantium
+Text Label 4000 1850 2    50   ~ 0
+Sensed28
+$Comp
+L Connector:TestPoint TP10
+U 1 1 5DC6EF69
+P 5350 2650
+F 0 "TP10" H 5408 2768 50  0000 L CNN
+F 1 "5V" H 5408 2677 50  0000 L CNN
+F 2 "TestPoint:TestPoint_Loop_D2.50mm_Drill1.0mm" H 5550 2650 50  0001 C CNN
+F 3 "~" H 5550 2650 50  0001 C CNN
+	1    5350 2650
+	1    0    0    -1
+$EndComp
+$Comp
+L Connector:TestPoint TP9
+U 1 1 5DC6FCB8
+P 4750 2650
+F 0 "TP9" H 4808 2768 50  0000 L CNN
+F 1 "5VRAW" H 4808 2677 50  0000 L CNN
+F 2 "TestPoint:TestPoint_Loop_D2.50mm_Drill1.0mm" H 4950 2650 50  0001 C CNN
+F 3 "~" H 4950 2650 50  0001 C CNN
+	1    4750 2650
+	1    0    0    -1
+$EndComp
+$Comp
+L Connector:TestPoint TP11
+U 1 1 5DC700AD
+P 6400 2650
+F 0 "TP11" H 6458 2768 50  0000 L CNN
+F 1 "3.3V" H 6458 2677 50  0000 L CNN
+F 2 "TestPoint:TestPoint_Loop_D2.50mm_Drill1.0mm" H 6600 2650 50  0001 C CNN
+F 3 "~" H 6600 2650 50  0001 C CNN
+	1    6400 2650
+	1    0    0    -1
+$EndComp
+Connection ~ 2700 3050
+$Comp
+L Connector:TestPoint TP8
+U 1 1 5DC6E713
+P 2700 3050
+F 0 "TP8" V 2895 3122 50  0000 C CNN
+F 1 "GND Loop" V 2804 3122 50  0000 C CNN
+F 2 "TestPoint:TestPoint_Loop_D2.50mm_Drill1.0mm" H 2900 3050 50  0001 C CNN
+F 3 "~" H 2900 3050 50  0001 C CNN
+	1    2700 3050
+	0    -1   -1   0
+$EndComp
+$Comp
+L Connector:TestPoint TP7
+U 1 1 5DC6E3A6
+P 2700 2250
+F 0 "TP7" H 2758 2368 50  0000 L CNN
+F 1 "28V Loop" H 2758 2277 50  0000 L CNN
+F 2 "TestPoint:TestPoint_Loop_D2.50mm_Drill1.0mm" H 2900 2250 50  0001 C CNN
+F 3 "~" H 2900 2250 50  0001 C CNN
+	1    2700 2250
+	1    0    0    -1
+$EndComp
 $EndSCHEMATC
